File: so40.kicad_sch (KiCad schematic)
At the start: 50 parts

Commit message: fuck ocean
Parts:
- removed J?: (no value), symbol kbd:MJ-4PP-9
- added D? (x3): D, Diodes_ThroughHole:Diode_DO-41_SOD81_Horizontal_RM10, symbol lets_split-rescue:D
- added J?: OLED, kbd:OLED, symbol Connector_Generic:Conn_01x04
- added J?: (no value), symbol kbd:MJ-4PP-9
- added JP? (x8): (no value), kbd:Jumper, symbol corne-classic-cache:Device{colon}Jumper_NO_Small
- added SW? (x3): SW_PUSH, flipalps:MXALPS_FLIP, symbol lets_split-rescue:SW_PUSH
Connections:
- net col3: now also SW?.1
- net col4: now also SW?.1
- net col5: now also SW?.1
- net row4: now reaches U?.11 (8/B4)
- net row4: now also D?.1 (K), D?.1 (K), D?.1 (K)
- net VCC: now reaches U?.21 (VCC)
- net VCC: now also J?.D, JP?.1, JP?.1
- net reset: now reaches U?.22 (RST)
- net GND: now reaches U?.23 (GND)
- net GND: now also U?.3 (GND), U?.4 (GND), J?.C, JP?.1, JP?.1
- net SDA: now reaches U?.5 (2/D1/SDA)
- net SDA: now also J?.A, JP?.1, JP?.1
- net SCL: now reaches U?.6 (3/D0/SCL)
- net SCL: now also J?.B, JP?.1, JP?.1
- new net: J?.1 (Pin_1), JP?.2, JP?.2
- new net: J?.2 (Pin_2), JP?.2, JP?.2
- new net: J?.4 (Pin_4), JP?.2, JP?.2
- new net: J?.3 (Pin_3), JP?.2, JP?.2
- new net: D?.2 (A), SW?.2 (x3)
- no-connect marks 0 -> 1
Other:
- moved on the sheet: D?, SW?

Commit message: done?
i think this is done
Parts:
- added J?: LED, kbd:StripLED_rev, symbol Connector_Generic:Conn_01x03
- added L? (x6): SK6812MINI, kbd:SK6812MINI_underglow, symbol kbd:SK6812MINI
- added L? (x27): SK6812MINI, kbd:SK6812MINI_rev, symbol kbd:SK6812MINI
- added R? (x2): R, kbd:R, symbol Device:R
- added RSW?: SW_PUSH, kbd:ResetSW, symbol corne-classic-cache:kbd{colon}SW_PUSH
Connections:
- net GND: now also J?.1 (Pin_1), L?.2 (VSS), L?.2 (VSS), L?.2 (VSS), L?.2 (VSS), L?.2 (VSS), L?.2 (VSS), L?.2 (VSS), L?.2 (VSS), L?.2 (VSS), L?.2 (VSS), L?.2 (VSS), L?.2 (VSS), L?.2 (VSS), L?.2 (VSS), L?.2 (VSS), L?.2 (VSS), L?.2 (VSS), L?.2 (VSS), L?.2 (VSS), L?.2 (VSS), L?.2 (VSS), L?.2 (VSS), L?.2 (VSS), L?.2 (VSS), L?.2 (VSS), RSW?.2
- net SCL: now also R?.2
- net SDA: now also R?.2
- net VCC: now also J?.3 (Pin_3), L?.4 (VDD), L?.4 (VDD), L?.4 (VDD), L?.4 (VDD), L?.4 (VDD), L?.4 (VDD), L?.4 (VDD), L?.4 (VDD), L?.4 (VDD), L?.4 (VDD), L?.4 (VDD), L?.4 (VDD), L?.4 (VDD), L?.4 (VDD), L?.4 (VDD), L?.4 (VDD), L?.4 (VDD), L?.4 (VDD), L?.4 (VDD), L?.4 (VDD), L?.4 (VDD), L?.4 (VDD), L?.4 (VDD), L?.4 (VDD), L?.4 (VDD), L?.4 (VDD), L?.4 (VDD), L?.4 (VDD), L?.4 (VDD), L?.4 (VDD), L?.4 (VDD), L?.4 (VDD), L?.4 (VDD), R?.1, R?.1
- net reset: now also RSW?.1
- net LED: now reaches U?.2 (RX1/D2)
- net LED: now also J?.2 (Pin_2), L?.3 (DIN)
- new net: L?.1 (DOUT), L?.3 (DIN) (x32)
- new net: L?.2 (VSS), L?.2 (VSS), L?.2 (VSS), L?.2 (VSS), L?.2 (VSS), L?.2 (VSS), L?.2 (VSS), L?.2 (VSS)
- no-connect marks 1 -> 4
Other:
- moved on the sheet: J?, JP?

Commit message: idk what i did
final touches to schematic, loaded footprints.
Parts:
- removed J?: (no value), symbol kbd:MJ-4PP-9
- added J1: SJ-43514, TRRS:CUI_SJ-43514, symbol trrs:SJ-43514
- D1, D10, D11, D12, D13, D14, D15, D16, D17, D18, D19, D2, D20, D21, D22, D23, D24, D25, D26, D27, D3, D4, D5, D6, D7, D8, D9: renamed from D?; footprint Diodes_ThroughHole:Diode_DO-41_SOD81_Horizontal_RM10 -> (none)
- L1, L2, L3, L4, L5, L6: renamed from L?; footprint kbd:SK6812MINI_underglow -> (none)
- SW1, SW10, SW11, SW12, SW13, SW14, SW15, SW16, SW17, SW18, SW19, SW2, SW20, SW21, SW22, SW23, SW24, SW25, SW26, SW27, SW3, SW4, SW5, SW6, SW7, SW8, SW9: renamed from SW?; footprint flipalps:MXALPS_FLIP -> (none)
- U1: renamed from U?; footprint (none) -> kbd:ProMicro_v2
- gave numbers to parts that had none: 40
Connections:
- net GND: now also J1.3
- net SCL: now also J1.4
- net SDA: now also J1.1
- net VCC: now also J1.2
- no-connect marks 4 -> 6

Commit message: before pcb
Parts:
- removed JP1, JP2, JP3, JP4, JP5, JP6, JP7, JP8: (no value), kbd:Jumper, symbol corne-classic-cache:Device{colon}Jumper_NO_Small
- D1, D10, D11, D12, D13, D14, D15, D16, D17, D18, D19, D2, D20, D21, D22, D23, D24, D25, D26, D27, D3, D4, D5, D6, D7, D8, D9: footprint (none) -> kbd:D3_TH_SMD
- L1, L2, L3, L4, L5, L6: footprint (none) -> kbd:SK6812MINI_underglow_rev
- SW1, SW10, SW11, SW12, SW13, SW14, SW15, SW16, SW17, SW18, SW19, SW2, SW20, SW21, SW22, SW23, SW24, SW25, SW26, SW27, SW3, SW4, SW5, SW6, SW7, SW8, SW9: footprint (none) -> kbd:MX_ALPS_PG1350_noLed
Connections:
- net SCL is gone; now on net VCC: J1.4, R2.2, U1.6 (3/D0/SCL)
- net SDA is gone; now on net GND: J1.1, R1.2, U1.5 (2/D1/SDA)
- net GND: now also J3.1 (Pin_1), J3.4 (Pin_4)
- net VCC: now also J3.2 (Pin_2), J3.3 (Pin_3)
